Commit message: Restructured the files

File: Inaccurate_Sketch/properties.xacro (robot description, xacro)
@@ -35,5 +35,5 @@
             <xacro:insert_block name="origin" />
             <mass value="${mass}" />
-            <inertia ixx="${(1/12) * mass * (3*radius*radius + length*length)" ixy="0.o" ixz="0.0"
+            <inertia ixx="${(1/12) * mass * (3*radius*radius + length*length)" ixy="0.0" ixz="0.0"
                     iyy="${(1/12) * mass * (3*radius*radius + length*length)]" iyz="0.0"
                     izz="${(1/2) * mass * (radius*radius)}" />
