Commit message: Renamed

File: urdf/simon.urdf (robot description, URDF)
Before this commit: robot four_DoF_manipulator, 6 links, 6 joints
Links:
- added link world
- link a1: mass 0.5 -> None
- link a2: mass 0.75 -> None
- link a3: mass 2.5 -> None
- link a4: mass 1.5 -> None
- link a5: mass 0.8 -> None
- link base_link: mass 10 -> None
