Commit message: Properly configured files

File: sw_exported_urdf/urdf/sw_exported_urdf.urdf (robot description, URDF)
Before this commit: robot ARM ASSEMBLY, 9 links, 8 joints
Links:
- removed link gripper_1
- removed link gripper_2
- added link link_gripper_1, mass 0.0075809; collision mesh filename=package://sw_exported_urdf/meshes/gripper_1.STL; visual mesh filename=package://sw_exported_urdf/meshes/gripper_1.STL
- added link link_gripper_2, mass 0.0081376; collision mesh filename=package://sw_exported_urdf/meshes/gripper_2.STL; visual mesh filename=package://sw_exported_urdf/meshes/gripper_2.STL
- added link world
- link base_link: geometry collision mesh filename=package://sw_exported_urdf/meshes/base_link.STL; visual mesh filename=package://sw_exported_urdf/meshes/base_link.STL
- link link_1: geometry collision mesh filename=package://sw_exported_urdf/meshes/link_1.STL; visual mesh filename=package://sw_exported_urdf/meshes/link_1.STL
- link link_2: geometry collision mesh filename=package://sw_exported_urdf/meshes/link_2.STL; visual mesh filename=package://sw_exported_urdf/meshes/link_2.STL
- link link_3: geometry collision mesh filename=package://sw_exported_urdf/meshes/link_3.STL; visual mesh filename=package://sw_exported_urdf/meshes/link_3.STL
- link link_4: geometry collision mesh filename=package://sw_exported_urdf/meshes/link_4.STL; visual mesh filename=package://sw_exported_urdf/meshes/link_4.STL
- link link_5: geometry collision mesh filename=package://sw_exported_urdf/meshes/link_5.STL; visual mesh filename=package://sw_exported_urdf/meshes/link_5.STL
- link link_6: geometry collision mesh filename=package://sw_exported_urdf/meshes/link_6.STL; visual mesh filename=package://sw_exported_urdf/meshes/link_6.STL
Joints:
- removed joint gripper_1
- removed joint gripper_2
- added joint base_joint: type fixed, parent world, child base_link, origin xyz=0.0 0.0 0.15 rpy=0 0 0
- added joint joint_gripper_1: type prismatic, parent link_6, child link_gripper_1, origin xyz=0.00037333 -0.008425 -0.064 rpy=3.1416 0 3.1416, axis -1 0 0, limit lower=0 upper=0.0381 effort=100 velocity=3
- added joint joint_gripper_2: type prismatic, parent link_6, child link_gripper_2, origin xyz=-0.012 0.007575 -0.064 rpy=3.1416 0 0, axis 1 0 0, limit lower=-0.0381 upper=0 effort=100 velocity=3
- joint joint_1: limit lower=0 upper=6.284 effort=300 velocity=3 -> lower=2.55 upper=5.7280 effort=300 velocity=3
- joint joint_2: limit lower=0 upper=3.142 effort=200 velocity=3 -> lower=-0.35 upper=3.5340 effort=200 velocity=3
- joint joint_3: limit lower=-4.713 upper=0 effort=200 velocity=3 -> lower=-0.0488 upper=5.2280 effort=200 velocity=3
- joint joint_4: limit lower=0 upper=6.284 effort=200 velocity=3 -> lower=-3.142 upper=3.142 effort=200 velocity=3
- joint joint_5: limit lower=0 upper=3.142 effort=200 velocity=3 -> lower=-3.764 upper=0.6419 effort=200 velocity=3
- joint joint_6: limit lower=0 upper=6.284 effort=200 velocity=3 -> lower=-3.142 upper=3.142 effort=200 velocity=3
